File: AK4432_PCM1863_breakout_board.kicad_sch (KiCad schematic)
At the start: 38 parts, among them J1 Conn_01x08_Pin, U1 PCM1863DBTR, U2 LD1117S33TR_SOT223, U3 AK4432VT, U4 SN74AVC1T45DCKR, U5 MIC5365-3.3YC5, U6 SN74LVC1G04DCKR, U7 SN74HC74DR, U8 LD1117S33TR_SOT223, Y2 ECS-2520MV-xxx-xx

Commit message: finished preliminary schematic, started laying out.
Parts:
- removed C13, C14: 1uF, Capacitor_SMD:C_0201_0603Metric_Pad0.64x0.40mm_HandSolder, symbol Device:C
- removed C15: 10uF, Capacitor_SMD:C_0805_2012Metric_Pad1.18x1.45mm_HandSolder, symbol Device:C
- removed JP3: Jumper_2_Bridged, Connector_PinHeader_2.54mm:PinHeader_1x02_P2.54mm_Vertical, symbol Jumper:Jumper_2_Bridged
- removed U4: SN74AVC1T45DCKR, DCK6, symbol SN74AVC1T45:SN74AVC1T45DCKR
- removed U5: MIC5365-3.3YC5, Package_TO_SOT_SMD:SOT-353_SC-70-5_Handsoldering, symbol Regulator_Linear:MIC5365-3.3YC5
- added C18, C22, C23: 1uF, Capacitor_SMD:C_0603_1608Metric_Pad1.08x0.95mm_HandSolder, symbol Device:C
- added C19: 2.2uF, Capacitor_SMD:C_0603_1608Metric_Pad1.08x0.95mm_HandSolder, symbol Device:C
- added C2, C21, C6: .1uF, Capacitor_SMD:C_0805_2012Metric_Pad1.18x1.45mm_HandSolder, symbol Device:C
- added C27: 10uF, Capacitor_SMD:C_0805_2012Metric_Pad1.18x1.45mm_HandSolder, symbol Device:C
- added J1, J7, J8: Conn_01x02_Pin, Connector_PinHeader_2.54mm:PinHeader_1x02_P2.54mm_Vertical, symbol Connector:Conn_01x02_Pin
- added J2, J3: Conn_01x04_Pin, Connector_PinHeader_2.54mm:PinHeader_1x04_P2.54mm_Vertical, symbol Connector:Conn_01x04_Pin
- added J5: Conn_01x07_Pin, Connector_PinHeader_2.54mm:PinHeader_1x07_P2.54mm_Vertical, symbol Connector:Conn_01x07_Pin
- added J6: Conn_01x01_Pin, Connector_PinHeader_2.54mm:PinHeader_1x01_P2.54mm_Vertical, symbol Connector:Conn_01x01_Pin
- added JP2: Jumper_2_Bridged, Connector_PinHeader_2.54mm:PinHeader_1x02_P2.54mm_Vertical, symbol Jumper:Jumper_2_Bridged
- added JP3: Jumper_3_Bridged12, Connector_PinHeader_2.54mm:PinHeader_1x03_P2.54mm_Vertical, symbol Jumper:Jumper_3_Bridged12
- added R1, R10, R11, R12, R13, R14, R15, R2, R3, R4, R5, R6, R7, R8, R9: 100, Resistor_SMD:R_0603_1608Metric_Pad0.98x0.95mm_HandSolder, symbol Device:R
- C20: value 1uF -> 10uF; footprint Capacitor_SMD:C_0201_0603Metric_Pad0.64x0.40mm_HandSolder -> Capacitor_SMD:C_0805_2012Metric_Pad1.18x1.45mm_HandSolder
- U3: renamed from U1; footprint footprints:DBT30_TEX -> footprints:DBT30_TEX-M
- U4: renamed from U3; footprint footprints:TSSOP16_AKM -> footprints:TSSOP16_AKM-M
- U5: renamed from U7; footprint D14 -> footprints:D14-M
- U6: footprint DCK0005A_N -> footprints:DCK0005A_M
- Y1: renamed from Y2; value ECS-2520MV-xxx-xx -> ECS-3225MV-491.52
- renumbered C2 to C1, C5 to C10, C6 to C11, C7 to C12, C8 to C13, C9 to C14, C10 to C15, C18 to C24, C19 to C25, C21 to C28, C22 to C29, C1 to C3, C23 to C5, C24 to C7, C25 to C8, C3 to C9, FB2 to FB1, J1 to J4, JP2 to JP1, R2 to R16, U2 to U1, U8 to U2
Connections:
- net 1.8V is gone; now on net GND: C20.2
- net +3.3_analog: now also C20.1, U4.14 (AVDD), C21.1
- net +3.3_digital: now also C26.2, U4.15 (LVDD), U6.5 (VCC), C27.2, JP2.2 (B), JP3.3 (B)
- net +5V: now also C2.1, C6.1, J1.1 (Pin_1)
- net GND: now also U4.13 (VSS), U4.9 (P/S), C18.2, C19.1, C2.2, C21.2, C27.1, C6.2, J1.2 (Pin_2), JP3.1 (A); no longer C20.1
- net GPIO1/INTA: now also R13.1
- net GPIO2/INTB: now also R14.1
- net GPIO3/INTC: now also R15.1
- net I2S_BCK: now also U4.2 (BICK), R6.1
- net I2S_LRCK: now also U4.4 (LRCK), R8.1
- net MICBIAS: now also J6.1 (Pin_1)
- net SCKI: now also U5.3 (1CLK), U6.4 (Y)
- net SPI_CS: now also R9.1
- net SPI_MISO: now also R12.1
- net SPI_MOSI: now also R11.1
- net SPI_SCLK: now also R10.1
- net at C25.2, FB1.2, R16.1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: no longer C26.2, U6.5 (VCC)
- net at U4.10 (AOUTR): now also C22.2, J7.1 (Pin_1)
- net at U4.11 (AOUTL): now also C23.2, J7.2 (Pin_2)
- net at U4.12 (VCOM): now also C19.2
- net at U4.16 (LDOO): now also C18.1
- net I2S_DIN_DAC: now reaches U4.3 (SDTI)
- net I2S_DIN_DAC: now also R7.1
- net AK_CS/I2CFIL: now reaches U4.6 (SMUTE/CSN/I2CFIL)
- net AK_CS/I2CFIL: now also JP3.2 (C), R2.2
- net ADC_PDN/RST renamed AK_PDN/RST
- net AK_PDN/RST: now also JP2.1 (A), R1.2
- net I2C_SCL renamed AK_SCL/CCLK
- net AK_SCL/CCLK: now also R3.2
- net I2C_SDA renamed AK_SDA/CDTI
- net AK_SDA/CDTI: now also R4.2
- net I2S_DOUT renamed I2S_DOUT_ADC
- net I2S_DOUT_ADC: now also R5.1
- net XI: no longer names the net of U3.10 (XI)
- new net: J2.1 (Pin_1), R1.1
- new net: J2.2 (Pin_2), R2.1
- new net: J2.3 (Pin_3), R3.1
- new net: J2.4 (Pin_4), R4.1
- new net: J3.2 (Pin_2), R6.2
- new net: J5.3 (Pin_3), R11.2
- new net: J3.1 (Pin_1), R5.2
- new net: J3.3 (Pin_3), R7.2
- new net: J3.4 (Pin_4), R8.2
- new net: J5.4 (Pin_4), R12.2
- new net: C22.1, J8.1 (Pin_1)
- new net: J5.2 (Pin_2), R10.2
- new net: J5.5 (Pin_5), R13.2
- new net: J5.6 (Pin_6), R14.2
- new net: J5.1 (Pin_1), R9.2
- new net: C23.1, J8.2 (Pin_2)
- new net: J5.7 (Pin_7), R15.2
- no-connect marks 4 -> 5
Other:
- note added: "USE 50V FOR THESE!"
- note removed: "(PCM Master Clock)"
- note removed: "1.8V regulator"
- note removed: "3.3V to 1.8V level shifter for PCM chip master clock"
- moved on the sheet: C1, C10, C11, C12, C13, C14, C15, C24, C25, C26, C28, C29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

Commit message: almost done laying out 2-layer prototype
Connections:
- net AK_CS/I2CFIL: no longer JP3.2 (C)
- net L1/1P: now also J4.6 (Pin_6); no longer J4.7 (Pin_7)
- net L2/1M: now also J4.8 (Pin_8); no longer J4.5 (Pin_5)
- net R1/2P: now also J4.5 (Pin_5); no longer J4.8 (Pin_8)
- net R2/2M: now also J4.7 (Pin_7); no longer J4.6 (Pin_6)
- net AK_CS/I2CFIL_R: now reaches J2.2 (Pin_2), R2.1
- net AK_CS/I2CFIL_R: now also JP3.2 (C)
Other:
- moved on the sheet: JP3
Changed lines of the file:
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@@
 	(text "(i2c)\nLo = 400kHz\nHi = 1MHz"
 		(exclude_from_sim no)
-		(at 73.914 181.102 0)
+		(at 52.324 177.292 0)
 		(effects
 			(font
@@
 	)
 	(junction
-		(at 73.66 173.99)
-		(diameter 0)
-		(color 0 0 0 0)
-	)
-	(junction
 		(at 354.33 52.07)
 		(diameter 0)
@@
 	)
 	(junction
+		(at 182.88 31.75)
+		(diameter 0)
+		(color 0 0 0 0)
+	)
+	(junction
 		(at 68.58 247.65)
 		(diameter 0)
@@
 	(wire
 		(pts
-			(xy 386.08 78.74) (xy 386.08 85.09)
+			(xy 180.34 200.66) (xy 182.88 200.66)
 		)
 		(stroke
@@
 	(wire
 		(pts
-			(xy 180.34 200.66) (xy 182.88 200.66)
+			(xy 68.58 247.65) (xy 82.55 247.65)
 		)
 		(stroke
@@
 	(wire
 		(pts
-			(xy 68.58 247.65) (xy 82.55 247.65)
+			(xy 146.05 49.53) (xy 146.05 45.72)
 		)
 		(stroke
@@
 	(wire
 		(pts
-			(xy 146.05 49.53) (xy 146.05 45.72)
+			(xy 71.12 135.89) (xy 77.47 135.89)
 		)
 		(stroke
@@
 	(wire
 		(pts
-			(xy 71.12 135.89) (xy 77.47 135.89)
+			(xy 354.33 39.37) (xy 354.33 41.91)
 		)
 		(stroke
@@
 	(wire
 		(pts
-			(xy 354.33 39.37) (xy 354.33 41.91)
+			(xy 391.16 82.55) (xy 391.16 78.74)
 		)
 		(stroke
@@
 	(wire
 		(pts
-			(xy 180.34 31.75) (xy 186.69 31.75)
+			(xy 180.34 31.75) (xy 182.88 31.75)
 		)
 		(stroke
@@
 	(wire
 		(pts
-			(xy 58.42 166.37) (xy 63.5 166.37)
+			(xy 36.83 162.56) (xy 41.91 162.56)
 		)
 		(stroke
@@
 	(wire
 		(pts
-			(xy 391.16 90.17) (xy 391.16 78.74)
-		)
-		(stroke
-			(width 0)
-			(type default)
-		)
-	)
-	(wire
-		(pts
 			(xy 281.94 88.9) (xy 281.94 90.17)
 		)
@@
 	(wire
 		(pts
+			(xy 386.08 87.63) (xy 386.08 78.74)
+		)
+		(stroke
+			(width 0)
+			(type default)
+		)
+	)
+	(wire
+		(pts
 			(xy 116.84 257.81) (xy 115.57 257.81)
 		)
@@
 	(wire
 		(pts
+			(xy 181.61 41.91) (xy 182.88 41.91)
+		)
+		(stroke
+			(width 0)
+			(type default)
+		)
+	)
+	(wire
+		(pts
 			(xy 393.7 52.07) (xy 381 52.07)
 		)
@@
 	(wire
 		(pts
-			(xy 388.62 78.74) (xy 388.62 87.63)
-		)
-		(stroke
-			(width 0)
-			(type default)
-		)
-	)
-	(wire
-		(pts
 			(xy 147.32 54.61) (xy 147.32 55.88)
 		)
@@
 	(wire
 		(pts
-			(xy 346.71 85.09) (xy 386.08 85.09)
+			(xy 346.71 85.09) (xy 388.62 85.09)
 		)
 		(stroke
@@
 	(wire
 		(pts
-			(xy 344.17 82.55) (xy 383.54 82.55)
+			(xy 344.17 82.55) (xy 391.16 82.55)
 		)
 		(stroke
@@
 	(wire
 		(pts
-			(xy 63.5 166.37) (xy 63.5 167.64)
+			(xy 41.91 162.56) (xy 41.91 163.83)
 		)
 		(stroke
@@
 	(wire
 		(pts
-			(xy 349.25 87.63) (xy 388.62 87.63)
+			(xy 349.25 87.63) (xy 386.08 87.63)
 		)
 		(stroke
@@
 	(wire
 		(pts
+			(xy 45.72 170.18) (xy 52.07 170.18)
+		)
+		(stroke
+			(width 0)
+			(type default)
+		)
+	)
+	(wire
+		(pts
 			(xy 161.29 52.07) (xy 166.37 52.07)
 		)
@@
 	(wire
 		(pts
+			(xy 383.54 90.17) (xy 383.54 78.74)
+		)
+		(stroke
+			(width 0)
+			(type default)
+		)
+	)
+	(wire
+		(pts
 			(xy 196.85 257.81) (xy 212.09 257.81)
 		)
@@
 	(wire
 		(pts
+			(xy 182.88 31.75) (xy 186.69 31.75)
+		)
+		(stroke
+			(width 0)
+			(type default)
+		)
+	)
+	(wire
+		(pts
 			(xy 172.72 260.35) (xy 172.72 262.89)
 		)
@@
 	(wire
 		(pts
+			(xy 388.62 85.09) (xy 388.62 78.74)
+		)
+		(stroke
+			(width 0)
+			(type default)
+		)
+	)
+	(wire
+		(pts
 			(xy 438.15 107.95) (xy 438.15 85.09)
 		)
@@
 	(wire
 		(pts
+			(xy 182.88 41.91) (xy 182.88 31.75)
+		)
+		(stroke
+			(width 0)
+			(type default)
+		)
+	)
+	(wire
+		(pts
 			(xy 175.26 68.58) (xy 184.15 68.58)
 		)
@@
 	(wire
 		(pts
-			(xy 351.79 90.17) (xy 391.16 90.17)
+			(xy 351.79 90.17) (xy 383.54 90.17)
 		)
 		(stroke
@@
 	(wire
 		(pts
-			(xy 67.31 173.99) (xy 73.66 173.99)
-		)
-		(stroke
-			(width 0)
-			(type default)
-		)
-	)
-	(wire
-		(pts
 			(xy 200.66 147.32) (xy 212.09 147.32)
 		)
@@
 	(wire
 		(pts
-			(xy 63.5 180.34) (xy 63.5 182.88)
+			(xy 41.91 176.53) (xy 41.91 179.07)
 		)
 		(stroke
@@
 		)
 	)
-	(wire
-		(pts
-			(xy 383.54 82.55) (xy 383.54 78.74)
-		)
-		(stroke
-			(width 0)
-			(type default)
-		)
-	)
 	(label "AK_CS{slash}I2CFIL"
 		(at 205.74 31.75 0)
@@
 		)
 	)
+	(label "AK_CS{slash}I2CFIL_R"
+		(at 181.61 41.91 180)
+		(effects
+			(font
+				(size 1.27 1.27)
+			)
+			(justify right bottom)
+		)
+	)
 	(label "I2S_LRCK"
 		(at 107.95 168.91 180)
@@
 		)
 	)
+	(label "AK_CS{slash}I2CFIL_R"
+		(at 52.07 170.18 0)
+		(effects
+			(font
+				(size 1.27 1.27)
+			)
+			(justify left bottom)
+		)
+	)
 	(label "SPI_MISO"
 		(at 433.07 123.19 0)
@@
 	)
 	(label "+3.3_digital"
-		(at 58.42 166.37 180)
+		(at 36.83 162.56 180)
 		(effects
 			(font
@@
 	(symbol
 		(lib_id "power:GND")
-		(at 63.5 182.88 0)
+		(at 41.91 179.07 0)
 		(unit 1)
 		(exclude_from_sim no)
@@
 		(fields_autoplaced yes)
 		(property "Reference" "#PWR013"
-			(at 63.5 189.23 0)
+			(at 41.91 185.42 0)
 			(effects
 				(font
@@
 		)
 		(property "Value" "GND"
-			(at 63.5 187.96 0)
+			(at 41.91 184.15 0)
 			(effects
 				(font
@@
 		)
 		(property "Footprint" ""
-			(at 63.5 182.88 0)
+			(at 41.91 179.07 0)
 			(effects
 				(font
@@
 		)
 		(property "Datasheet" ""
-			(at 63.5 182.88 0)
+			(at 41.91 179.07 0)
 			(effects
 				(font
@@
 		)
 		(property "Description" "Power symbol creates a global label with name \"GND\" , ground"
-			(at 63.5 182.88 0)
+			(at 41.91 179.07 0)
 			(effects
 				(font
@@
 	(symbol
 		(lib_id "Jumper:Jumper_3_Bridged12")
-		(at 63.5 173.99 90)
+		(at 41.91 170.18 90)
 		(unit 1)
 		(exclude_from_sim no)
@@
 		(dnp no)
 		(property "Reference" "JP3"
-			(at 65.278 170.18 90)
+			(at 43.688 166.37 90)
 			(effects
 				(font
@@
 		)
 		(property "Value" "Jumper_3_Bridged12"
-			(at 65.024 175.768 90)
+			(at 43.434 171.958 90)
 			(effects
 				(font
@@
 		)
 		(property "Footprint" "Connector_PinHeader_2.54mm:PinHeader_1x03_P2.54mm_Vertical"
-			(at 63.5 173.99 0)
+			(at 41.91 170.18 0)
 			(effects
 				(font
@@
 		)
 		(property "Datasheet" "~"
-			(at 63.5 173.99 0)
+			(at 41.91 170.18 0)
 			(effects
 				(font
@@
 		)
 		(property "Description" "Jumper, 3-pole, pins 1+2 closed/bridged"
-			(at 63.5 173.99 0)
+			(at 41.91 170.18 0)
 			(effects
 				(font

Commit message: finished 2 layer layoutgit add -A
Parts:
- removed C1, C5: 100uF, Capacitor_THT:CP_Radial_D6.3mm_P2.50mm, symbol Device:C
- added C1, C5: 100uF, Capacitor_THT:CP_Radial_D6.3mm_P2.50mm, symbol Device:C_Polarized
Connections:
- net +5V: now also C1.1, C5.1
- net GND: now also C1.2, C5.2
- net L1/1P renamed L1_1P
- net L2/1M renamed L2_1M
- net L3/4P renamed L3_4P
- net L4/4M renamed L4_4M
- net R1/2P renamed R1_2P
- net R2/2M renamed R2_2M
- net R3/3P renamed R3_3P
- net R4/3M renamed R4_3M
Changed lines of the file:
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@@
 		)
 	)
-	(label "R1{slash}2P"
+	(label "R1_2P"
 		(at 377.19 82.55 180)
 		(effects
@@
 		)
 	)
-	(label "L4{slash}4M"
+	(label "L4_4M"
 		(at 407.67 82.55 0)
 		(effects
@@
 		)
 	)
-	(label "L1{slash}1P"
+	(label "L1_1P"
 		(at 378.46 85.09 180)
 		(effects
@@
 		)
 	)
-	(label "L3{slash}4P"
+	(label "L3_4P"
 		(at 405.13 87.63 0)
 		(effects
@@
 		)
 	)
-	(label "R4{slash}3M"
+	(label "R4_3M"
 		(at 406.4 85.09 0)
 		(effects
@@
 		)
 	)
-	(label "R2{slash}2M"
+	(label "R2_2M"
 		(at 379.73 87.63 180)
 		(effects
@@
 		)
 	)
-	(label "L2{slash}1M"
+	(label "L2_1M"
 		(at 381 90.17 180)
 		(effects
@@
 		)
 	)
-	(label "R3{slash}3P"
+	(label "R3_3P"
 		(at 403.86 90.17 0)
 		(effects
@@
 	)
 	(symbol
-		(lib_id "Device:C")
-		(at 237.49 40.64 0)
-		(unit 1)
-		(exclude_from_sim no)
-		(in_bom yes)
-		(on_board yes)
-		(dnp no)
-		(fields_autoplaced yes)
-		(property "Reference" "C1"
-			(at 241.3 39.3699 0)
-			(effects
-				(font
-					(size 1.27 1.27)
-				)
-				(justify left)
-			)
-		)
-		(property "Value" "100uF"
-			(at 241.3 41.9099 0)
-			(effects
-				(font
-					(size 1.27 1.27)
-				)
-				(justify left)
-			)
-		)
-		(property "Footprint" "Capacitor_THT:CP_Radial_D6.3mm_P2.50mm"
-			(at 238.4552 44.45 0)
-			(effects
-				(font
-					(size 1.27 1.27)
-				)
-				(hide yes)
-			)
-		)
-		(property "Datasheet" "~"
-			(at 237.49 40.64 0)
-			(effects
-				(font
-					(size 1.27 1.27)
-				)
-				(hide yes)
-			)
-		)
-		(property "Description" "Unpolarized capacitor"
-			(at 237.49 40.64 0)
-			(effects
-				(font
-					(size 1.27 1.27)
-				)
-				(hide yes)
-			)
-		)
-		(pin "2"
-		)
-		(pin "1"
-		)
-		(instances
-			(project "AK4432_PCM1863_breakout_board"
-				(path "/8c03b016-3db6-4507-be73-495931c2d93e"
-					(reference "C1")
-					(unit 1)
-				)
-			)
-		)
-	)
-	(symbol
 		(lib_id "Connector:Conn_01x04_Pin")
 		(at 171.45 52.07 0)
@@
 	)
 	(symbol
-		(lib_id "Device:C")
-		(at 341.63 45.72 0)
-		(unit 1)
-		(exclude_from_sim no)
-		(in_bom yes)
-		(on_board yes)
-		(dnp no)
-		(fields_autoplaced yes)
-		(property "Reference" "C5"
-			(at 345.44 44.4499 0)
-			(effects
-				(font
-					(size 1.27 1.27)
-				)
-				(justify left)
-			)
-		)
-		(property "Value" "100uF"
-			(at 345.44 46.9899 0)
-			(effects
-				(font
-					(size 1.27 1.27)
-				)
-				(justify left)
-			)
-		)
-		(property "Footprint" "Capacitor_THT:CP_Radial_D6.3mm_P2.50mm"
-			(at 342.5952 49.53 0)
-			(effects
-				(font
-					(size 1.27 1.27)
-				)
-				(hide yes)
-			)
-		)
-		(property "Datasheet" "~"
-			(at 341.63 45.72 0)
-			(effects
-				(font
-					(size 1.27 1.27)
-				)
-				(hide yes)
-			)
-		)
-		(property "Description" "Unpolarized capacitor"
-			(at 341.63 45.72 0)
-			(effects
-				(font
-					(size 1.27 1.27)
-				)
-				(hide yes)
-			)
-		)
-		(pin "2"
-		)
-		(pin "1"
-		)
-		(instances
-			(project "AK4432_PCM1863_breakout_board"
-				(path "/8c03b016-3db6-4507-be73-495931c2d93e"
-					(reference "C5")
-					(unit 1)
-				)
-			)
-		)
-	)
-	(symbol
 		(lib_id "Jumper:Jumper_2_Bridged")
 		(at 66.04 135.89 0)
@@
 	)
 	(symbol
+		(lib_id "Device:C_Polarized")
+		(at 341.63 45.72 0)
+		(unit 1)
+		(exclude_from_sim no)
+		(in_bom yes)
+		(on_board yes)
+		(dnp no)
+		(fields_autoplaced yes)
+		(property "Reference" "C5"
+			(at 345.44 43.5609 0)
+			(effects
+				(font
+					(size 1.27 1.27)
+				)
+				(justify left)
+			)
+		)
+		(property "Value" "100uF"
+			(at 345.44 46.1009 0)
+			(effects
+				(font
+					(size 1.27 1.27)
+				)
+				(justify left)
+			)
+		)
+		(property "Footprint" "Capacitor_THT:CP_Radial_D6.3mm_P2.50mm"
+			(at 342.5952 49.53 0)
+			(effects
+				(font
+					(size 1.27 1.27)
+				)
+				(hide yes)
+			)
+		)
+		(property "Datasheet" "~"
+			(at 341.63 45.72 0)
+			(effects
+				(font
+					(size 1.27 1.27)
+				)
+				(hide yes)
+			)
+		)
+		(property "Description" "Polarized capacitor"
+			(at 341.63 45.72 0)
+			(effects
+				(font
+					(size 1.27 1.27)
+				)
+				(hide yes)
+			)
+		)
+		(pin "2"
+		)
+		(pin "1"
+		)
+		(instances
+			(project "AK4432_PCM1863_breakout_board"
+				(path "/8c03b016-3db6-4507-be73-495931c2d93e"
+					(reference "C5")
+					(unit 1)
+				)
+			)
+		)
+	)
+	(symbol
 		(lib_id "power:PWR_FLAG")
 		(at 134.62 22.86 0)
@@
 					(unit 1)
 				)
+			)
+		)
+	)
+	(symbol
+		(lib_id "Device:C_Polarized")
+		(at 237.49 40.64 0)
+		(unit 1)
+		(exclude_from_sim no)
+		(in_bom yes)
+		(on_board yes)
+		(dnp no)
+		(fields_autoplaced yes)
+		(property "Reference" "C1"
+			(at 241.3 38.4809 0)
+			(effects
+				(font
+					(size 1.27 1.27)
+				)
+				(justify left)
+			)
+		)
+		(property "Value" "100uF"
+			(at 241.3 41.0209 0)
+			(effects
+				(font
+					(size 1.27 1.27)
+				)
+				(justify left)
+			)
+		)
+		(property "Footprint" "Capacitor_THT:CP_Radial_D6.3mm_P2.50mm"
+			(at 238.4552 44.45 0)
+			(effects
+				(font
+					(size 1.27 1.27)
+				)
+				(hide yes)
+			)
+		)
+		(property "Datasheet" "~"
+			(at 237.49 40.64 0)
+			(effects
+				(font
+					(size 1.27 1.27)
+				)
+				(hide yes)
+			)
+		)
+		(property "Description" "Polarized capacitor"
+			(at 237.49 40.64 0)
+			(effects
+				(font
+					(size 1.27 1.27)
+				)
+				(hide yes)
+			)
+		)
+		(pin "2"
+		)
+		(pin "1"
+		)
+		(instances
+			(project ""
+				(path "/8c03b016-3db6-4507-be73-495931c2d93e"
+					(reference "C1")
+					(unit 1)
+				)

Commit message: Finished v1 layout! Also swaped flip-flop chip for a faster one.
Parts:
- removed C1: 100uF, Capacitor_THT:CP_Radial_D6.3mm_P2.50mm, symbol Device:C_Polarized
- removed U5: SN74HC74DR, footprints:D14-M, symbol SN74HC74DR_flip-flop:SN74HC74DR
- added H1, H2, H3: MountingHole, MountingHole:MountingHole_3.2mm_M3, symbol Mechanical:MountingHole
- added U5: SN74LVC1G74DCUR, DCU0008A_N, symbol SN74LVC1G74DCUR-flip-flop:SN74LVC1G74DCUR
- renumbered C2 to C1, C11 to C10, C12 to C11, C13 to C12, C14 to C13, C15 to C14, C16 to C15, C17 to C16, C18 to C17, C19 to C18, C20 to C19, C3 to C2, C21 to C20, C22 to C21, C23 to C22, C24 to C23, C25 to C24, C26 to C25, C27 to C26, C28 to C27, C29 to C28, C4 to C3, C5 to C4, C6 to C5, C7 to C6, C8 to C7, C9 to C8, C10 to C9
Connections:
- net +3.3_digital: now also U5.6 (CLR_N), U5.7 (PRE_N), U5.8 (VCC)
- net GND: now also U5.4 (GND)
- net MCLK_AKM: now also U5.5 (Q)
- net SCKI: now also U5.1 (CLK)
- net PWR_RST: now reaches J2.1 (Pin_1), R1.1
- net SCL_CCLK: now reaches J2.3 (Pin_3), R3.1
- net SDA_CDTI: now reaches J2.4 (Pin_4), R4.1
- net BCK: now reaches J3.2 (Pin_2), R6.2
- net MOSI: now reaches J5.3 (Pin_3), R11.2
- net DOUT_ADC: now reaches J3.1 (Pin_1), R5.2
- net DIN_DAC: now reaches J3.3 (Pin_3), R7.2
- net LRCK: now reaches J3.4 (Pin_4), R8.2
- net MISO: now reaches J5.4 (Pin_4), R12.2
- net DAC_OUTR: now reaches C21.2, J7.1 (Pin_1), U4.10 (AOUTR)
- net SCLK: now reaches J5.2 (Pin_2), R10.2
- net DAC_OUTL: now reaches C22.2, J7.2 (Pin_2), U4.11 (AOUTL)
- net 1_A: now reaches J5.5 (Pin_5), R13.2
- net 2_B: now reaches J5.6 (Pin_6), R14.2
- net CS: now reaches J5.1 (Pin_1), R9.2
- net 3_C: now reaches J5.7 (Pin_7), R15.2
- net AK_CS/I2CFIL renamed AK_CS_I2CFIL
- net AK_CS/I2CFIL_R renamed CS_I2CFreq
- net AK_PDN/RST renamed AK_PD_RST
- net AK_SCL/CCLK renamed AK_SCL_CCLK
- net AK_SDA/CDTI renamed AK_SDA_CDTI
- net GPIO1/INTA renamed GPIO1_INTA
- net GPIO2/INTB renamed GPIO2_INTB
- net GPIO3/INTC renamed GPIO3_INTC
- new net: U5.2 (D), U5.3 (Q_N)
- no-connect marks 5 -> 3
Other:
- moved on the sheet: C27, C28, J2, J3, J5
